File: hardware/shop-output-board/shop-output-board.kicad_pcb (KiCad board)
At the start: 2 copper layers, 150 x 115 mm, 84 parts

Commit message: regenerate the v1 board, gerbers and schematic for both fixes
Carries the 1812 polyfuse and the LED polarity correction into the routed board and the fab
outputs. The board is hand-routed and cannot be regenerated, so both changes were applied to
it surgically:

  F1  - footprint swapped 1206 -> 1812, pads move from +/-1.4 to +/-2.1375, and the VIN_RAW
        and VIN_F traces extended 0.7375mm to meet them. Without that the old endpoints sat
        0.175mm outside the new pads and would have read as unconnected. Nearest neighbour is
        8.5mm away, so the larger body cost nothing in layout.
  LED - pad nets swapped and the footprint rotated 180, which changes no copper.

DRC is clean at 0 violations and 0 unconnected. Pad positions verified against KiCad's own
IPC-D-356 export; the only mismatch it reports is D9, which was rotated 180 by hand during
routing and is expected - rotation preserves pin-to-net mapping.

The stale upload zip is dropped rather than refreshed. It wrapped the pre-1812 Gerbers, and
the tracked Gerber folder is the thing that matters.

Co-Authored-By: Claude Opus 5 <noreply@anthropic.com>
Parts:
- F1: footprint Fuse:Fuse_1206_3216Metric -> Fuse:Fuse_1812_4532Metric
- turned LED1 to 180 degrees
- turned LED2 to 180 degrees
- turned LED3 to 180 degrees
- turned LED4 to 180 degrees
- turned LED5 to 180 degrees
- turned LED6 to 180 degrees
- turned LED7 to 180 degrees
- turned LED8 to 180 degrees
Connections:
- LED1 pad 1: LEDK1 -> ISO_GND
- LED1 pad 2: ISO_GND -> LEDK1
- LED2 pad 1: LEDK2 -> ISO_GND
- LED2 pad 2: ISO_GND -> LEDK2
- LED3 pad 1: LEDK3 -> ISO_GND
- LED3 pad 2: ISO_GND -> LEDK3
- LED4 pad 1: LEDK4 -> ISO_GND
- LED4 pad 2: ISO_GND -> LEDK4
- LED5 pad 1: LEDK5 -> ISO_GND
- LED5 pad 2: ISO_GND -> LEDK5
- LED6 pad 1: LEDK6 -> ISO_GND
- LED6 pad 2: ISO_GND -> LEDK6
- LED7 pad 1: LEDK7 -> ISO_GND
- LED7 pad 2: ISO_GND -> LEDK7
- LED8 pad 1: LEDK8 -> ISO_GND
- LED8 pad 2: ISO_GND -> LEDK8
Routing:
- net VIN_RAW: track 19.5 -> 18.8 mm
- net VIN_F: track 9.54 -> 8.80 mm
Changed lines of the file:
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@@
 		)
 	)
-	(footprint "Fuse:Fuse_1206_3216Metric"
+	(footprint "Fuse:Fuse_1812_4532Metric"
 		(layer "F.Cu")
-		(at 28 92)
-		(descr "Fuse SMD 1206 (3216 Metric), square (rectangular) end terminal, IPC-7351 nominal, (Body size source: http://www.tortai-tech.com/upload/download/2011102023233369053.pdf)")
+		(at 28.0 92.0)
+		(descr "Fuse SMD 1812 (4532 Metric), square (rectangular) end terminal, IPC-7351 nominal, (Body size source: https://www.nikhef.nl/pub/departments/mt/projects/detectorR_D/dtddice/ERJ2G.pdf)")
 		(tags "fuse")
 		(property "Reference" "F1"
-			(at 0 -2 0)
+			(at 0 -2.65 0)
 			(layer "F.SilkS")
 			(effects
@@
 		(duplicate_pad_numbers_are_jumpers no)
 		(fp_line
-			(start -0.602064 -0.91)
-			(end 0.602064 -0.91)
+			(start -1.386252 -1.71)
+			(end 1.386252 -1.71)
 			(stroke
 				(width 0.12)
@@
 		)
 		(fp_line
-			(start -0.602064 0.91)
-			(end 0.602064 0.91)
+			(start -1.386252 1.71)
+			(end 1.386252 1.71)
 			(stroke
 				(width 0.12)
@@
 		)
 		(fp_rect
-			(start -2.28 -1.13)
-			(end 2.28 1.13)
+			(start -2.95 -1.95)
+			(end 2.95 1.95)
 			(stroke
 				(width 0.05)
@@
 		)
 		(fp_rect
-			(start -1.6 -0.8)
-			(end 1.6 0.8)
+			(start -2.25 -1.6)
+			(end 2.25 1.6)
 			(stroke
 				(width 0.1)
@@
 		)
 		(pad "1" smd roundrect
-			(at -1.4 0)
-			(size 1.25 1.75)
+			(at -2.1375 0)
+			(size 1.125 3.4)
 			(layers "F.Cu" "F.Mask" "F.Paste")
-			(roundrect_rratio 0.2)
+			(roundrect_rratio 0.222222)
 			(net "VIN_RAW")
 		)
 		(pad "2" smd roundrect
-			(at 1.4 0)
-			(size 1.25 1.75)
+			(at 2.1375 0)
+			(size 1.125 3.4)
 			(layers "F.Cu" "F.Mask" "F.Paste")
-			(roundrect_rratio 0.2)
+			(roundrect_rratio 0.222222)
 			(net "VIN_F")
 		)
 		(embedded_fonts no)
-		(model "${KICAD10_3DMODEL_DIR}/Fuse.3dshapes/Fuse_1206_3216Metric.step"
+		(model "${KICAD10_3DMODEL_DIR}/Fuse.3dshapes/Fuse_1812_4532Metric.step"
 			(offset
 				(xyz 0 0 0)
@@
 	(footprint "LED_SMD:LED_0805_2012Metric"
 		(layer "F.Cu")
-		(at 15 80)
+		(at 15 80 180)
 		(descr "LED SMD 0805 (2012 Metric), square (rectangular) end terminal, IPC-7351 nominal, (Body size source: https://docs.google.com/spreadsheets/d/1BsfQQcO9C6DZCsRaXUlFlo91Tg2WpOkGARC1WS5S8t0/edit?usp=sharing)")
 		(tags "LED")
@@
 		)
 		(pad "1" smd roundrect
-			(at -0.9375 0)
+			(at -0.9375 0 180)
 			(size 0.975 1.4)
 			(layers "F.Cu" "F.Mask" "F.Paste")
 			(roundrect_rratio 0.25)
-			(net "LEDK1")
+			(net "ISO_GND")
 		)
 		(pad "2" smd roundrect
-			(at 0.9375 0)
+			(at 0.9375 0 180)
 			(size 0.975 1.4)
 			(layers "F.Cu" "F.Mask" "F.Paste")
 			(roundrect_rratio 0.25)
-			(net "ISO_GND")
+			(net "LEDK1")
 		)
 		(embedded_fonts no)
@@
 	(footprint "LED_SMD:LED_0805_2012Metric"
 		(layer "F.Cu")
-		(at 127 80)
+		(at 127 80 180)
 		(descr "LED SMD 0805 (2012 Metric), square (rectangular) end terminal, IPC-7351 nominal, (Body size source: https://docs.google.com/spreadsheets/d/1BsfQQcO9C6DZCsRaXUlFlo91Tg2WpOkGARC1WS5S8t0/edit?usp=sharing)")
 		(tags "LED")
@@
 		)
 		(pad "1" smd roundrect
-			(at -0.9375 0)
+			(at -0.9375 0 180)
 			(size 0.975 1.4)
 			(layers "F.Cu" "F.Mask" "F.Paste")
 			(roundrect_rratio 0.25)
-			(net "LEDK8")
+			(net "ISO_GND")
 		)
 		(pad "2" smd roundrect
-			(at 0.9375 0)
+			(at 0.9375 0 180)
 			(size 0.975 1.4)
 			(layers "F.Cu" "F.Mask" "F.Paste")
 			(roundrect_rratio 0.25)
-			(net "ISO_GND")
+			(net "LEDK8")
 		)
 		(embedded_fonts no)
@@
 	(footprint "LED_SMD:LED_0805_2012Metric"
 		(layer "F.Cu")
-		(at 111 80)
+		(at 111 80 180)
 		(descr "LED SMD 0805 (2012 Metric), square (rectangular) end terminal, IPC-7351 nominal, (Body size source: https://docs.google.com/spreadsheets/d/1BsfQQcO9C6DZCsRaXUlFlo91Tg2WpOkGARC1WS5S8t0/edit?usp=sharing)")
 		(tags "LED")
@@
 		)
 		(pad "1" smd roundrect
-			(at -0.9375 0)
+			(at -0.9375 0 180)
 			(size 0.975 1.4)
 			(layers "F.Cu" "F.Mask" "F.Paste")
 			(roundrect_rratio 0.25)
-			(net "LEDK7")
+			(net "ISO_GND")
 		)
 		(pad "2" smd roundrect
-			(at 0.9375 0)
+			(at 0.9375 0 180)
 			(size 0.975 1.4)
 			(layers "F.Cu" "F.Mask" "F.Paste")
 			(roundrect_rratio 0.25)
-			(net "ISO_GND")
+			(net "LEDK7")
 		)
 		(embedded_fonts no)
@@
 	(footprint "LED_SMD:LED_0805_2012Metric"
 		(layer "F.Cu")
-		(at 31 80)
+		(at 31 80 180)
 		(descr "LED SMD 0805 (2012 Metric), square (rectangular) end terminal, IPC-7351 nominal, (Body size source: https://docs.google.com/spreadsheets/d/1BsfQQcO9C6DZCsRaXUlFlo91Tg2WpOkGARC1WS5S8t0/edit?usp=sharing)")
 		(tags "LED")
@@
 		)
 		(pad "1" smd roundrect
-			(at -0.9375 0)
+			(at -0.9375 0 180)
 			(size 0.975 1.4)
 			(layers "F.Cu" "F.Mask" "F.Paste")
 			(roundrect_rratio 0.25)
-			(net "LEDK2")
+			(net "ISO_GND")
 		)
 		(pad "2" smd roundrect
-			(at 0.9375 0)
+			(at 0.9375 0 180)
 			(size 0.975 1.4)
 			(layers "F.Cu" "F.Mask" "F.Paste")
 			(roundrect_rratio 0.25)
-			(net "ISO_GND")
+			(net "LEDK2")
 		)
 		(embedded_fonts no)
@@
 	(footprint "LED_SMD:LED_0805_2012Metric"
 		(layer "F.Cu")
-		(at 63 80)
+		(at 63 80 180)
 		(descr "LED SMD 0805 (2012 Metric), square (rectangular) end terminal, IPC-7351 nominal, (Body size source: https://docs.google.com/spreadsheets/d/1BsfQQcO9C6DZCsRaXUlFlo91Tg2WpOkGARC1WS5S8t0/edit?usp=sharing)")
 		(tags "LED")
@@
 		)
 		(pad "1" smd roundrect
-			(at -0.9375 0)
+			(at -0.9375 0 180)
 			(size 0.975 1.4)
 			(layers "F.Cu" "F.Mask" "F.Paste")
 			(roundrect_rratio 0.25)
-			(net "LEDK4")
+			(net "ISO_GND")
 		)
 		(pad "2" smd roundrect
-			(at 0.9375 0)
+			(at 0.9375 0 180)
 			(size 0.975 1.4)
 			(layers "F.Cu" "F.Mask" "F.Paste")
 			(roundrect_rratio 0.25)
-			(net "ISO_GND")
+			(net "LEDK4")
 		)
 		(embedded_fonts no)
@@
 	(footprint "LED_SMD:LED_0805_2012Metric"
 		(layer "F.Cu")
-		(at 47 80)
+		(at 47 80 180)
 		(descr "LED SMD 0805 (2012 Metric), square (rectangular) end terminal, IPC-7351 nominal, (Body size source: https://docs.google.com/spreadsheets/d/1BsfQQcO9C6DZCsRaXUlFlo91Tg2WpOkGARC1WS5S8t0/edit?usp=sharing)")
 		(tags "LED")
@@
 		)
 		(pad "1" smd roundrect
-			(at -0.9375 0)
+			(at -0.9375 0 180)
 			(size 0.975 1.4)
 			(layers "F.Cu" "F.Mask" "F.Paste")
 			(roundrect_rratio 0.25)
-			(net "LEDK3")
+			(net "ISO_GND")
 		)
 		(pad "2" smd roundrect
-			(at 0.9375 0)
+			(at 0.9375 0 180)
 			(size 0.975 1.4)
 			(layers "F.Cu" "F.Mask" "F.Paste")
 			(roundrect_rratio 0.25)
-			(net "ISO_GND")
+			(net "LEDK3")
 		)
 		(embedded_fonts no)
@@
 	(footprint "LED_SMD:LED_0805_2012Metric"
 		(layer "F.Cu")
-		(at 95 80)
+		(at 95 80 180)
 		(descr "LED SMD 0805 (2012 Metric), square (rectangular) end terminal, IPC-7351 nominal, (Body size source: https://docs.google.com/spreadsheets/d/1BsfQQcO9C6DZCsRaXUlFlo91Tg2WpOkGARC1WS5S8t0/edit?usp=sharing)")
 		(tags "LED")
@@
 		)
 		(pad "1" smd roundrect
-			(at -0.9375 0)
+			(at -0.9375 0 180)
 			(size 0.975 1.4)
 			(layers "F.Cu" "F.Mask" "F.Paste")
 			(roundrect_rratio 0.25)
-			(net "LEDK6")
+			(net "ISO_GND")
 		)
 		(pad "2" smd roundrect
-			(at 0.9375 0)
+			(at 0.9375 0 180)
 			(size 0.975 1.4)
 			(layers "F.Cu" "F.Mask" "F.Paste")
 			(roundrect_rratio 0.25)
-			(net "ISO_GND")
+			(net "LEDK6")
 		)
 		(embedded_fonts no)
@@
 	(footprint "LED_SMD:LED_0805_2012Metric"
 		(layer "F.Cu")
-		(at 79 80)
+		(at 79 80 180)
 		(descr "LED SMD 0805 (2012 Metric), square (rectangular) end terminal, IPC-7351 nominal, (Body size source: https://docs.google.com/spreadsheets/d/1BsfQQcO9C6DZCsRaXUlFlo91Tg2WpOkGARC1WS5S8t0/edit?usp=sharing)")
 		(tags "LED")
@@
 		)
 		(pad "1" smd roundrect
-			(at -0.9375 0)
+			(at -0.9375 0 180)
 			(size 0.975 1.4)
 			(layers "F.Cu" "F.Mask" "F.Paste")
 			(roundrect_rratio 0.25)
-			(net "LEDK5")
+			(net "ISO_GND")
 		)
 		(pad "2" smd roundrect
-			(at 0.9375 0)
+			(at 0.9375 0 180)
 			(size 0.975 1.4)
 			(layers "F.Cu" "F.Mask" "F.Paste")
 			(roundrect_rratio 0.25)
-			(net "ISO_GND")
+			(net "LEDK5")
 		)
 		(embedded_fonts no)
@@
 	(segment
 		(start 38.9375 92)
-		(end 29.4 92)
+		(end 30.1375 92)
 		(width 0.2)
 		(layer "F.Cu")
@@
 	)
 	(segment
-		(start 26.6 92)
+		(start 25.8625 92)
 		(end 19.55 92)
 		(width 0.2)
