File: hardware/shop-output-board/shop-output-board.kicad_sch (KiCad schematic)
At the start: 84 parts, among them J1 V+ IN 5-24V, J2 OUT 1-4, J3 OUT 5-8, J4 Pico 1-20, J5 Pico 21-40, Q1 AO3401A, Q2 AO3401A, Q3 AO3401A, Q4 AO3401A, Q5 AO3401A, Q6 AO3401A, Q7 AO3401A, Q8 AO3401A, Q9 reverse-polarity, U1 PC817B, U2 PC817B, U3 PC817B, U4 PC817B, U5 PC817B, U6 PC817B, U7 PC817B, U8 PC817B

Commit message: assign footprints, and swap two parts so pins map to pads
Every symbol now carries a footprint, checked automatically: the file exists on
disk and has a pad for every pin the netlist uses.

Two part changes came out of that check rather than from preference.

The MOSFETs were Device:Q_PMOS, whose pins are numbered G/D/S. Footprint pads
are named 1/2/3, so the board would have imported with every transistor
unconnected. Now the real Transistor_FET:AO3401A, which inherits 1=G, 2=S, 3=D
from its parent and matches the physical SOT-23. The generator resolves the
extends chain so the schematic stays self-contained.

The Zeners were specified as BZX84C8V2 in SOT-23 - a three-pad package for a
two-pin symbol, same class of mismatch. Now MMSZ5237B in SOD-123.

Q9 becomes an AO3401A as well. At 4A it has ample margin over the whole board's
draw and it collapses the BOM to a single MOSFET line.

The opto is DIP-4 rather than the SMD option on purpose: the wider body buys
creepage across the isolation barrier, the one place on this board where
spacing is load-bearing.

verify_netlist.py caught the pin renaming immediately when the MOSFET symbol
changed, which is what it is for.

kicad-cli sch erc: 0 violations. 78 nets, 84 parts, all assertions pass.

Co-Authored-By: Claude Opus 5 <noreply@anthropic.com>
Parts:
- C1: footprint (none) -> Capacitor_SMD:CP_Elec_8x10.5
- C2: footprint (none) -> Capacitor_SMD:C_0805_2012Metric
- D1, D2, D3, D4, D5, D6, D7, D8, D9: value BZX84C8V2 -> MMSZ5237B 8V2; footprint (none) -> Diode_SMD:D_SOD-123
- F1: footprint (none) -> Fuse:Fuse_1206_3216Metric
- J1: footprint (none) -> TerminalBlock_Phoenix:TerminalBlock_Phoenix_MKDS-1,5-2-5.08_1x02_P5.08mm_Horizontal
- J2, J3: footprint (none) -> TerminalBlock_Phoenix:TerminalBlock_Phoenix_MKDS-1-6-3.81_1x06_P3.81mm_Horizontal
- J4, J5: footprint (none) -> Connector_PinSocket_2.54mm:PinSocket_1x20_P2.54mm_Vertical
- LED1, LED2, LED3, LED4, LED5, LED6, LED7, LED8: footprint (none) -> LED_SMD:LED_0805_2012Metric
- Q1, Q2, Q3, Q4, Q5, Q6, Q7, Q8: footprint (none) -> Package_TO_SOT_SMD:SOT-23; symbol Device:Q_PMOS -> Transistor_FET:AO3401A
- Q9: value reverse-polarity -> AO3401A; footprint (none) -> Package_TO_SOT_SMD:SOT-23; symbol Device:Q_PMOS -> Transistor_FET:AO3401A
- R101, R102, R103, R104, R105, R201, R202, R203, R204, R205, R301, R302, R303, R304, R305, R401, R402, R403, R404, R405, R501, R502, R503, R504, R505, R6, R601, R602, R603, R604, R605, R701, R702, R703, R704, R705, R801, R802, R803, R804, R805: footprint (none) -> Resistor_SMD:R_0805_2012Metric
- TVS1: footprint (none) -> Diode_SMD:D_SMA
- U1, U2, U3, U4, U5, U6, U7, U8: footprint (none) -> Package_DIP:DIP-4_W7.62mm
Connections:
- net GATE1: now also Q1.1 (G); no longer Q1.G
- net GATE2: now also Q2.1 (G); no longer Q2.G
- net GATE3: now also Q3.1 (G); no longer Q3.G
- net GATE4: now also Q4.1 (G); no longer Q4.G
- net GATE5: now also Q5.1 (G); no longer Q5.G
- net GATE6: now also Q6.1 (G); no longer Q6.G
- net GATE7: now also Q7.1 (G); no longer Q7.G
- net GATE8: now also Q8.1 (G); no longer Q8.G
- net OUT1: now also Q1.3 (D); no longer Q1.D
- net OUT2: now also Q2.3 (D); no longer Q2.D
- net OUT3: now also Q3.3 (D); no longer Q3.D
- net OUT4: now also Q4.3 (D); no longer Q4.D
- net OUT5: now also Q5.3 (D); no longer Q5.D
- net OUT6: now also Q6.3 (D); no longer Q6.D
- net OUT7: now also Q7.3 (D); no longer Q7.D
- net OUT8: now also Q8.3 (D); no longer Q8.D
- net Q9GATE: now also Q9.1 (G); no longer Q9.G
- net V+: now also Q1.2 (S), Q2.2 (S), Q3.2 (S), Q4.2 (S), Q5.2 (S), Q6.2 (S), Q7.2 (S), Q8.2 (S), Q9.2 (S); no longer Q1.S, Q2.S, Q3.S, Q4.S, Q5.S, Q6.S, Q7.S, Q8.S, Q9.S
- net VIN_F: now also Q9.3 (D); no longer Q9.D

Commit message: switch the optocoupler to SMD so the board suits partial assembly
Moving to SMT assembly with hand-soldered connectors left the DIP-4
optocouplers as the only through-hole part a machine would otherwise want to
place. Switched to the gull-wing SOP-4 version.

This improves the barrier rather than compromising it, which was not obvious
going in. SOP-4 leads splay outward to a 9.38mm pad row span against the DIP-4's
7.62mm, so the 5mm barrier now has 1.39mm of pad clearance instead of 0.51mm.
The package would allow a gap up to 7.8mm; the extra clearance is worth more
than a wider gap, since 5mm already far exceeds what 24V functional isolation
needs.

The board is now 79 SMD parts and 5 through-hole - the three screw terminals
and two Pico socket strips, which is exactly the split between what a machine
finds awkward and a person finds easy.

Fabrication guide rewritten around the three assembly options, with the
position-file flag that excludes through-hole parts, and a sequence that avoids
paying assembly charges on an unproven board: breadboard a channel, then bare
boards to prove the layout, then the assembled run.

ERC still 0 violations, 78 nets, all assertions pass.

Co-Authored-By: Claude Opus 5 <noreply@anthropic.com>
Parts:
- U1, U2, U3, U4, U5, U6, U7, U8: value PC817B -> LTV-817S (CTR B); footprint Package_DIP:DIP-4_W7.62mm -> Package_SO:SOP-4_7.5x4.1mm_P2.54mm
Changed lines of the file:
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@@
 			)
 		)
-		(property "Value" "PC817B"
+		(property "Value" "LTV-817S (CTR B)"
 			(at 36.83 90.17 0)
 			(effects
@@
 			)
 		)
-		(property "Footprint" "Package_DIP:DIP-4_W7.62mm"
+		(property "Footprint" "Package_SO:SOP-4_7.5x4.1mm_P2.54mm"
 			(at 30.48 90.17 0)
 			(hide yes)
@@
 			)
 		)
-		(property "Value" "PC817B"
+		(property "Value" "LTV-817S (CTR B)"
 			(at 104.14 90.17 0)
 			(effects
@@
 			)
 		)
-		(property "Footprint" "Package_DIP:DIP-4_W7.62mm"
+		(property "Footprint" "Package_SO:SOP-4_7.5x4.1mm_P2.54mm"
 			(at 97.79 90.17 0)
 			(hide yes)
@@
 			)
 		)
-		(property "Value" "PC817B"
+		(property "Value" "LTV-817S (CTR B)"
 			(at 172.72 90.17 0)
 			(effects
@@
 			)
 		)
-		(property "Footprint" "Package_DIP:DIP-4_W7.62mm"
+		(property "Footprint" "Package_SO:SOP-4_7.5x4.1mm_P2.54mm"
 			(at 166.37 90.17 0)
 			(hide yes)
@@
 			)
 		)
-		(property "Value" "PC817B"
+		(property "Value" "LTV-817S (CTR B)"
 			(at 240.03 90.17 0)
 			(effects
@@
 			)
 		)
-		(property "Footprint" "Package_DIP:DIP-4_W7.62mm"
+		(property "Footprint" "Package_SO:SOP-4_7.5x4.1mm_P2.54mm"
 			(at 233.68 90.17 0)
 			(hide yes)
@@
 			)
 		)
-		(property "Value" "PC817B"
+		(property "Value" "LTV-817S (CTR B)"
 			(at 308.61 90.17 0)
 			(effects
@@
 			)
 		)
-		(property "Footprint" "Package_DIP:DIP-4_W7.62mm"
+		(property "Footprint" "Package_SO:SOP-4_7.5x4.1mm_P2.54mm"
 			(at 302.26 90.17 0)
 			(hide yes)
@@
 			)
 		)
-		(property "Value" "PC817B"
+		(property "Value" "LTV-817S (CTR B)"
 			(at 375.92 90.17 0)
 			(effects
@@
 			)
 		)
-		(property "Footprint" "Package_DIP:DIP-4_W7.62mm"
+		(property "Footprint" "Package_SO:SOP-4_7.5x4.1mm_P2.54mm"
 			(at 369.57 90.17 0)
 			(hide yes)
@@
 			)
 		)
-		(property "Value" "PC817B"
+		(property "Value" "LTV-817S (CTR B)"
 			(at 444.5 90.17 0)
 			(effects
@@
 			)
 		)
-		(property "Footprint" "Package_DIP:DIP-4_W7.62mm"
+		(property "Footprint" "Package_SO:SOP-4_7.5x4.1mm_P2.54mm"
 			(at 438.15 90.17 0)
 			(hide yes)
@@
 			)
 		)
-		(property "Value" "PC817B"
+		(property "Value" "LTV-817S (CTR B)"
 			(at 511.81 90.17 0)
 			(effects
@@
 			)
 		)
-		(property "Footprint" "Package_DIP:DIP-4_W7.62mm"
+		(property "Footprint" "Package_SO:SOP-4_7.5x4.1mm_P2.54mm"
 			(at 505.46 90.17 0)
 			(hide yes)

Commit message: put manufacturer part numbers in the BOM
"100k" is not orderable. Every line now carries an MPN and manufacturer,
emitted as schematic fields so the BOM export picks them up rather than being
maintained separately and drifting.

Two entries carry requirements that are easy to lose to a well-meaning
substitution, so the reason is written next to them: the optocoupler must be
CTR rank B or the opto cannot sink R2's current from 4.5mA of LED drive, and
the indicator LED wants a high-efficiency part because it runs at about 1.4mA
on a 5V supply.

None of these have been checked against live distributor stock, which the
comment says plainly. Suffixes for tape, tolerance and CTR rank vary by
packaging and want confirming with whoever assembles the board.

F1 is deliberately left as VERIFY. A polyfuse's voltage rating is what it can
interrupt when it trips, many 1206 parts are rated 6V or 16V, and this rail
reaches 24V - a part that fails instead of opening is worse than no part. The
options are written up in design.md; it is flagged rather than fixed because
changing the footprint would invalidate Gerbers that are already exported.

ERC 0, netlist assertions pass, 78 nets, 84 parts unchanged.

Co-Authored-By: Claude Opus 5 <noreply@anthropic.com>
Parts:
- C1: MPN (none) -> EEE-FK1H101P; Manufacturer (none) -> Panasonic
- C2: MPN (none) -> CL21B104KBCNNNC; Manufacturer (none) -> Samsung
- D1, D2, D3, D4, D5, D6, D7, D8, D9: MPN (none) -> MMSZ5237B-7-F; Manufacturer (none) -> Diodes Inc
- F1: MPN (none) -> VERIFY - see design.md; Manufacturer (none) -> -
- J1: MPN (none) -> 1729128; Manufacturer (none) -> Phoenix Contact
- J2, J3: MPN (none) -> 1727010; Manufacturer (none) -> Phoenix Contact
- J4, J5: MPN (none) -> PPTC201LFBN-RC; Manufacturer (none) -> Sullins
- LED1, LED2, LED3, LED4, LED5, LED6, LED7, LED8: MPN (none) -> LTST-C170KGKT; Manufacturer (none) -> Lite-On
- Q1, Q2, Q3, Q4, Q5, Q6, Q7, Q8, Q9: MPN (none) -> AO3401A; Manufacturer (none) -> Alpha & Omega
- R101, R201, R301, R401, R501, R6, R601, R701, R801: MPN (none) -> RC0805FR-07100KL; Manufacturer (none) -> Yageo
- R102, R202, R302, R402, R502, R602, R702, R802: MPN (none) -> RC0805FR-074K7L; Manufacturer (none) -> Yageo
- R103, R203, R303, R403, R503, R603, R703, R803: MPN (none) -> RC0805FR-0710KL; Manufacturer (none) -> Yageo
- R104, R204, R304, R404, R504, R604, R704, R804: MPN (none) -> RC0805FR-072K2L; Manufacturer (none) -> Yageo
- R105, R205, R305, R405, R505, R605, R705, R805: MPN (none) -> RC0805FR-07470RL; Manufacturer (none) -> Yageo
- TVS1: MPN (none) -> SMAJ30A; Manufacturer (none) -> Littelfuse
- U1, U2, U3, U4, U5, U6, U7, U8: MPN (none) -> LTV-817S-TA1-B; Manufacturer (none) -> Lite-On

Commit message: regenerate the v1 board, gerbers and schematic for both fixes
Carries the 1812 polyfuse and the LED polarity correction into the routed board and the fab
outputs. The board is hand-routed and cannot be regenerated, so both changes were applied to
it surgically:

  F1  - footprint swapped 1206 -> 1812, pads move from +/-1.4 to +/-2.1375, and the VIN_RAW
        and VIN_F traces extended 0.7375mm to meet them. Without that the old endpoints sat
        0.175mm outside the new pads and would have read as unconnected. Nearest neighbour is
        8.5mm away, so the larger body cost nothing in layout.
  LED - pad nets swapped and the footprint rotated 180, which changes no copper.

DRC is clean at 0 violations and 0 unconnected. Pad positions verified against KiCad's own
IPC-D-356 export; the only mismatch it reports is D9, which was rotated 180 by hand during
routing and is expected - rotation preserves pin-to-net mapping.

The stale upload zip is dropped rather than refreshed. It wrapped the pre-1812 Gerbers, and
the tracked Gerber folder is the thing that matters.

Co-Authored-By: Claude Opus 5 <noreply@anthropic.com>
Parts:
- F1: footprint Fuse:Fuse_1206_3216Metric -> Fuse:Fuse_1812_4532Metric; MPN VERIFY - see design.md -> MF-MSMF110/24X-2; Manufacturer - -> Bourns
- J2, J3: MPN 1727010 -> 1727052
Connections:
- net ISO_GND: now also LED1.1 (K), LED2.1 (K), LED3.1 (K), LED4.1 (K), LED5.1 (K), LED6.1 (K), LED7.1 (K), LED8.1 (K); no longer LED1.2 (A), LED2.2 (A), LED3.2 (A), LED4.2 (A), LED5.2 (A), LED6.2 (A), LED7.2 (A), LED8.2 (A)
- net LEDK1: now also LED1.2 (A); no longer LED1.1 (K)
- net LEDK2: now also LED2.2 (A); no longer LED2.1 (K)
- net LEDK3: now also LED3.2 (A); no longer LED3.1 (K)
- net LEDK4: now also LED4.2 (A); no longer LED4.1 (K)
- net LEDK5: now also LED5.2 (A); no longer LED5.1 (K)
- net LEDK6: now also LED6.2 (A); no longer LED6.1 (K)
- net LEDK7: now also LED7.2 (A); no longer LED7.1 (K)
- net LEDK8: now also LED8.2 (A); no longer LED8.1 (K)
Changed lines of the file:
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@@
 	(wire
 		(pts
-			(xy 50.8 180.34) (xy 50.8 177.8)
+			(xy 58.42 180.34) (xy 58.42 177.8)
 		)
 		(stroke
@@
 	)
 	(label "LEDK1"
-		(at 50.8 177.8 90)
+		(at 58.42 177.8 90)
 		(effects
 			(font
@@
 	(wire
 		(pts
-			(xy 58.42 180.34) (xy 58.42 182.88)
+			(xy 50.8 180.34) (xy 50.8 182.88)
 		)
 		(stroke
@@
 	)
 	(label "ISO_GND"
-		(at 58.42 182.88 90)
+		(at 50.8 182.88 90)
 		(effects
 			(font
@@
 	(wire
 		(pts
-			(xy 119.38 180.34) (xy 119.38 177.8)
+			(xy 127.0 180.34) (xy 127.0 177.8)
 		)
 		(stroke
@@
 	)
 	(label "LEDK2"
-		(at 119.38 177.8 90)
+		(at 127.0 177.8 90)
 		(effects
 			(font
@@
 	(wire
 		(pts
-			(xy 127.0 180.34) (xy 127.0 182.88)
+			(xy 119.38 180.34) (xy 119.38 182.88)
 		)
 		(stroke
@@
 	)
 	(label "ISO_GND"
-		(at 127.0 182.88 90)
+		(at 119.38 182.88 90)
 		(effects
 			(font
@@
 	(wire
 		(pts
-			(xy 186.69 180.34) (xy 186.69 177.8)
+			(xy 194.31 180.34) (xy 194.31 177.8)
 		)
 		(stroke
@@
 	)
 	(label "LEDK3"
-		(at 186.69 177.8 90)
+		(at 194.31 177.8 90)
 		(effects
 			(font
@@
 	(wire
 		(pts
-			(xy 194.31 180.34) (xy 194.31 182.88)
+			(xy 186.69 180.34) (xy 186.69 182.88)
 		)
 		(stroke
@@
 	)
 	(label "ISO_GND"
-		(at 194.31 182.88 90)
+		(at 186.69 182.88 90)
 		(effects
 			(font
@@
 	(wire
 		(pts
-			(xy 255.27 180.34) (xy 255.27 177.8)
+			(xy 262.89 180.34) (xy 262.89 177.8)
 		)
 		(stroke
@@
 	)
 	(label "LEDK4"
-		(at 255.27 177.8 90)
+		(at 262.89 177.8 90)
 		(effects
 			(font
@@
 	(wire
 		(pts
-			(xy 262.89 180.34) (xy 262.89 182.88)
+			(xy 255.27 180.34) (xy 255.27 182.88)
 		)
 		(stroke
@@
 	)
 	(label "ISO_GND"
-		(at 262.89 182.88 90)
+		(at 255.27 182.88 90)
 		(effects
 			(font
@@
 	(wire
 		(pts
-			(xy 322.58 180.34) (xy 322.58 177.8)
+			(xy 330.2 180.34) (xy 330.2 177.8)
 		)
 		(stroke
@@
 	)
 	(label "LEDK5"
-		(at 322.58 177.8 90)
+		(at 330.2 177.8 90)
 		(effects
 			(font
@@
 	(wire
 		(pts
-			(xy 330.2 180.34) (xy 330.2 182.88)
+			(xy 322.58 180.34) (xy 322.58 182.88)
 		)
 		(stroke
@@
 	)
 	(label "ISO_GND"
-		(at 330.2 182.88 90)
+		(at 322.58 182.88 90)
 		(effects
 			(font
@@
 	(wire
 		(pts
-			(xy 391.16 180.34) (xy 391.16 177.8)
+			(xy 398.78 180.34) (xy 398.78 177.8)
 		)
 		(stroke
@@
 	)
 	(label "LEDK6"
-		(at 391.16 177.8 90)
+		(at 398.78 177.8 90)
 		(effects
 			(font
@@
 	(wire
 		(pts
-			(xy 398.78 180.34) (xy 398.78 182.88)
+			(xy 391.16 180.34) (xy 391.16 182.88)
 		)
 		(stroke
@@
 	)
 	(label "ISO_GND"
-		(at 398.78 182.88 90)
+		(at 391.16 182.88 90)
 		(effects
 			(font
@@
 	(wire
 		(pts
-			(xy 459.74 180.34) (xy 459.74 177.8)
+			(xy 467.36 180.34) (xy 467.36 177.8)
 		)
 		(stroke
@@
 	)
 	(label "LEDK7"
-		(at 459.74 177.8 90)
+		(at 467.36 177.8 90)
 		(effects
 			(font
@@
 	(wire
 		(pts
-			(xy 467.36 180.34) (xy 467.36 182.88)
+			(xy 459.74 180.34) (xy 459.74 182.88)
 		)
 		(stroke
@@
 	)
 	(label "ISO_GND"
-		(at 467.36 182.88 90)
+		(at 459.74 182.88 90)
 		(effects
 			(font
@@
 	(wire
 		(pts
-			(xy 527.05 180.34) (xy 527.05 177.8)
+			(xy 534.67 180.34) (xy 534.67 177.8)
 		)
 		(stroke
@@
 	)
 	(label "LEDK8"
-		(at 527.05 177.8 90)
+		(at 534.67 177.8 90)
 		(effects
 			(font
@@
 	(wire
 		(pts
-			(xy 534.67 180.34) (xy 534.67 182.88)
+			(xy 527.05 180.34) (xy 527.05 182.88)
 		)
 		(stroke
@@
 	)
 	(label "ISO_GND"
-		(at 534.67 182.88 90)
+		(at 527.05 182.88 90)
 		(effects
 			(font
@@
 			)
 		)
-		(property "Footprint" "Fuse:Fuse_1206_3216Metric"
+		(property "Footprint" "Fuse:Fuse_1812_4532Metric"
 			(at 69.85 234.95 0)
 			(hide yes)
@@
 			)
 		)
-		(property "MPN" "VERIFY - see design.md"
+		(property "MPN" "MF-MSMF110/24X-2"
 			(at 69.85 234.95 0)
 			(hide yes)
@@
 			)
 		)
-		(property "Manufacturer" "-"
+		(property "Manufacturer" "Bourns"
 			(at 69.85 234.95 0)
 			(hide yes)
@@
 			)
 		)
-		(property "MPN" "1727010"
+		(property "MPN" "1727052"
 			(at 320.04 234.95 0)
 			(hide yes)
@@
 			)
 		)
-		(property "MPN" "1727010"
+		(property "MPN" "1727052"
 			(at 379.73 234.95 0)
 			(hide yes)
